File: MFG/HP_device/HP_device.sch (KiCad schematic (older format))
At the start: 48 parts, among them J1 Screw_Terminal_01x02, J10 Screw_Terminal_01x02, J11 Screw_Terminal_01x02, J12 Screw_Terminal_01x02, J13 Screw_Terminal_01x02, J14 Screw_Terminal_01x02, J2 Screw_Terminal_01x02, J3 Screw_Terminal_01x02, J4 Screw_Terminal_01x02, J5 Screw_Terminal_01x02, J6 Screw_Terminal_01x02, J7 Screw_Terminal_01x02, J8 Screw_Terminal_01x02, J9 Screw_Terminal_01x02, K1 G5V-1, K2 G5V-1, K3 G5V-1, K4 G5V-1, K5 G5V-1, K6 G5V-1, Q1 BS170, Q2 BS170, Q3 BS170, Q4 BS170, Q5 BS170, Q6 BS170, Q7 BS170, U1 AT89C4051-24PU, U2 MCP4162-104, U3 MCP4162-503, U4 74HC595, U5 SN65176BP, U6 4N25, U7 4N25, U8 4N25, U9 4N25, Y1 Crystal

Commit message: Add layouts
Parts:
- added C3: C, Capacitor_THT:CP_Radial_D10.0mm_P5.00mm, symbol Device:C
- added D1: D, Diode_THT:D_5W_P12.70mm_Horizontal, symbol Device:D
- C1, C2: footprint (none) -> Capacitor_THT:C_Disc_D3.8mm_W2.6mm_P2.50mm
- J1, J10, J11, J12, J13, J14, J2, J3, J4, J5, J6, J7, J8, J9: footprint (none) -> TerminalBlock_Phoenix:TerminalBlock_Phoenix_MKDS-1,5-2_1x02_P5.00mm_Horizontal
- R1, R2, R3, R4, R5, R6, R7, R8: footprint (none) -> Resistor_THT:R_Axial_DIN0204_L3.6mm_D1.6mm_P5.08mm_Horizontal
- U2, U3: footprint (none) -> Package_DIP:DIP-8_W7.62mm
- U4: footprint (none) -> Package_DIP:DIP-16_W7.62mm
- Y1: footprint (none) -> Crystal:Crystal_HC18-U_Vertical
Connections:
- net +5V: now also C3.1, D1.1 (K); no longer J2.2 (Pin_2)
- net GND: now also C3.2
- new net: D1.2 (A), J2.2 (Pin_2)
Other:
- moved on the sheet: J2

Commit message: HP device scheamtic complete with footprints
Parts:
- added D2, D3, D4: TVSS, Diode_THT:D_A-405_P10.16mm_Horizontal, symbol Device:D
- added R9: 150, Resistor_THT:R_Axial_DIN0204_L3.6mm_D1.6mm_P5.08mm_Horizontal, symbol Device:R_Small
- C1, C2: value C -> 30p
- C3: footprint Capacitor_THT:CP_Radial_D10.0mm_P5.00mm -> Capacitor_THT:C_Radial_D6.3mm_H11.0mm_P2.50mm
- D1: footprint Diode_THT:D_5W_P12.70mm_Horizontal -> Diode_THT:D_A-405_P10.16mm_Horizontal
- R2: footprint Resistor_THT:R_Axial_DIN0204_L3.6mm_D1.6mm_P5.08mm_Horizontal -> Resistor_THT:R_Axial_DIN0309_L9.0mm_D3.2mm_P15.24mm_Horizontal
- R3, R4: value R_Small -> 200k; footprint Resistor_THT:R_Axial_DIN0204_L3.6mm_D1.6mm_P5.08mm_Horizontal -> Resistor_THT:R_Axial_DIN0309_L9.0mm_D3.2mm_P15.24mm_Horizontal
- R5: value R_Small -> 200K; footprint Resistor_THT:R_Axial_DIN0204_L3.6mm_D1.6mm_P5.08mm_Horizontal -> Resistor_THT:R_Axial_DIN0309_L9.0mm_D3.2mm_P15.24mm_Horizontal
- Y1: footprint Crystal:Crystal_HC18-U_Vertical -> Crystal:Crystal_HC49-4H_Vertical
Connections:
- net GND: now also D3.1 (K), D4.1 (K)
- net at J1.1 (Pin_1), U5.6 (A): now also D2.1 (K), D3.2 (A), D4.2 (A), R9.1
- net at J1.2 (Pin_2), U5.7 (B): now also D2.2 (A), R9.2
Other:
- moved on the sheet: J1, U5
Changed lines of the file:
@@
 F 0 "R2" V 2504 5400 50  0000 C CNN
 F 1 "200k" V 2595 5400 50  0000 C CNN
-F 2 "Resistor_THT:R_Axial_DIN0204_L3.6mm_D1.6mm_P5.08mm_Horizontal" H 2700 5400 50  0001 C CNN
+F 2 "Resistor_THT:R_Axial_DIN0309_L9.0mm_D3.2mm_P15.24mm_Horizontal" H 2700 5400 50  0001 C CNN
 F 3 "~" H 2700 5400 50  0001 C CNN
 	1    2700 5400
@@
 P 2700 5950
 F 0 "R3" V 2504 5950 50  0000 C CNN
-F 1 "R_Small" V 2595 5950 50  0000 C CNN
-F 2 "Resistor_THT:R_Axial_DIN0204_L3.6mm_D1.6mm_P5.08mm_Horizontal" H 2700 5950 50  0001 C CNN
+F 1 "200k" V 2595 5950 50  0000 C CNN
+F 2 "Resistor_THT:R_Axial_DIN0309_L9.0mm_D3.2mm_P15.24mm_Horizontal" H 2700 5950 50  0001 C CNN
 F 3 "~" H 2700 5950 50  0001 C CNN
 	1    2700 5950
@@
 P 2700 6500
 F 0 "R4" V 2504 6500 50  0000 C CNN
-F 1 "R_Small" V 2595 6500 50  0000 C CNN
-F 2 "Resistor_THT:R_Axial_DIN0204_L3.6mm_D1.6mm_P5.08mm_Horizontal" H 2700 6500 50  0001 C CNN
+F 1 "200k" V 2595 6500 50  0000 C CNN
+F 2 "Resistor_THT:R_Axial_DIN0309_L9.0mm_D3.2mm_P15.24mm_Horizontal" H 2700 6500 50  0001 C CNN
 F 3 "~" H 2700 6500 50  0001 C CNN
 	1    2700 6500
@@
 P 2700 7050
 F 0 "R5" V 2504 7050 50  0000 C CNN
-F 1 "R_Small" V 2595 7050 50  0000 C CNN
-F 2 "Resistor_THT:R_Axial_DIN0204_L3.6mm_D1.6mm_P5.08mm_Horizontal" H 2700 7050 50  0001 C CNN
+F 1 "200K" V 2595 7050 50  0000 C CNN
+F 2 "Resistor_THT:R_Axial_DIN0309_L9.0mm_D3.2mm_P15.24mm_Horizontal" H 2700 7050 50  0001 C CNN
 F 3 "~" H 2700 7050 50  0001 C CNN
 	1    2700 7050
@@
 L Connector:Screw_Terminal_01x02 J1
 U 1 1 63B3486B
-P 1200 3000
-F 0 "J1" H 1150 3100 50  0000 L CNN
-F 1 "Screw_Terminal_01x02" H 1280 2901 50  0001 L CNN
-F 2 "TerminalBlock_Phoenix:TerminalBlock_Phoenix_MKDS-1,5-2_1x02_P5.00mm_Horizontal" H 1200 3000 50  0001 C CNN
-F 3 "~" H 1200 3000 50  0001 C CNN
-	1    1200 3000
+P 650 2700
+F 0 "J1" H 600 2800 50  0000 L CNN
+F 1 "Screw_Terminal_01x02" H 730 2601 50  0001 L CNN
+F 2 "TerminalBlock_Phoenix:TerminalBlock_Phoenix_MKDS-1,5-2_1x02_P5.00mm_Horizontal" H 650 2700 50  0001 C CNN
+F 3 "~" H 650 2700 50  0001 C CNN
+	1    650  2700
 	-1   0    0    1
 $EndComp
@@
 L RS485Device:SN65176BP U5
 U 1 1 63BDC577
-P 2550 2950
-F 0 "U5" H 2550 3531 50  0000 C CNN
-F 1 "SN65176BP" H 2550 3440 50  0000 C CNN
-F 2 "Package_DIP:DIP-8_W7.62mm" H 2550 2450 50  0001 C CNN
-F 3 "https://www.ti.com/lit/ds/symlink/sn65176b.pdf" H 2550 2950 50  0001 C CNN
-	1    2550 2950
+P 2550 2500
+F 0 "U5" H 2550 3081 50  0000 C CNN
+F 1 "SN65176BP" H 2550 2990 50  0000 C CNN
+F 2 "Package_DIP:DIP-8_W7.62mm" H 2550 2000 50  0001 C CNN
+F 3 "https://www.ti.com/lit/ds/symlink/sn65176b.pdf" H 2550 2500 50  0001 C CNN
+	1    2550 2500
 	1    0    0    -1
 $EndComp
@@
 Text GLabel 6150 4150 2    50   Input ~ 0
 DRIVE
-Text GLabel 3300 2750 2    50   Input ~ 0
+Text GLabel 3300 2300 2    50   Input ~ 0
 RXD
-Text GLabel 3300 2850 2    50   Input ~ 0
+Text GLabel 3300 2400 2    50   Input ~ 0
 TXD
-Text GLabel 3300 3100 2    50   Input ~ 0
+Text GLabel 3300 2650 2    50   Input ~ 0
 DRIVE
 Wire Wire Line
-	3050 2750 3300 2750
-Wire Wire Line
-	3050 2850 3300 2850
-Wire Wire Line
-	3300 3100 3150 3100
-Wire Wire Line
-	3150 3100 3150 3050
-Wire Wire Line
-	3150 3050 3050 3050
-Wire Wire Line
-	3050 3150 3150 3150
-Wire Wire Line
-	3150 3150 3150 3100
-Connection ~ 3150 3100
-Wire Wire Line
-	1400 2900 1700 2900
-Wire Wire Line
-	1700 2900 1700 2850
-Wire Wire Line
-	1700 2850 2050 2850
-Wire Wire Line
-	2050 3050 1700 3050
-Wire Wire Line
-	1700 3050 1700 3000
-Wire Wire Line
-	1700 3000 1400 3000
-Wire Notes Line
-	700  2250 1750 2250
-Wire Notes Line
-	1750 2250 1750 4500
-Wire Notes Line
-	1750 4500 600  4500
-Text Notes 800  2450 0    50   ~ 0
+	3050 2300 3300 2300
+Wire Wire Line
+	3050 2400 3300 2400
+Wire Wire Line
+	3300 2650 3150 2650
+Wire Wire Line
+	3150 2650 3150 2600
+Wire Wire Line
+	3150 2600 3050 2600
+Wire Wire Line
+	3050 2700 3150 2700
+Wire Wire Line
+	3150 2700 3150 2650
+Connection ~ 3150 2650
+Text Notes 800  2050 0    50   ~ 0
 CONTROL & POWER
-Text Notes 650  2950 0    50   ~ 0
+Text Notes 550  2500 0    50   ~ 0
 RS485 Bus
 Text Notes 600  3400 0    50   ~ 0
@@
 F 0 "Y1" V 4404 3481 50  0000 L CNN
 F 1 "Crystal" V 4495 3481 50  0000 L CNN
-F 2 "Crystal:Crystal_HC18-U_Vertical" H 4450 3350 50  0001 C CNN
+F 2 "Crystal:Crystal_HC49-4H_Vertical" H 4450 3350 50  0001 C CNN
 F 3 "~" H 4450 3350 50  0001 C CNN
 	1    4450 3350
@@
 U 1 1 63CC4E89
 P 3850 3650
-F 0 "C1" H 3965 3696 50  0000 L CNN
-F 1 "C" H 3965 3605 50  0000 L CNN
+F 0 "C1" H 3650 3700 50  0000 L CNN
+F 1 "30p" H 3600 3600 50  0000 L CNN
 F 2 "Capacitor_THT:C_Disc_D3.8mm_W2.6mm_P2.50mm" H 3888 3500 50  0001 C CNN
 F 3 "~" H 3850 3650 50  0001 C CNN
@@
 P 4150 3650
 F 0 "C2" H 4265 3696 50  0000 L CNN
-F 1 "C" H 4265 3605 50  0000 L CNN
+F 1 "30p" H 4265 3605 50  0000 L CNN
 F 2 "Capacitor_THT:C_Disc_D3.8mm_W2.6mm_P2.50mm" H 4188 3500 50  0001 C CNN
 F 3 "~" H 4150 3650 50  0001 C CNN
@@
 L power:+5V #PWR0115
 U 1 1 63D739E3
-P 2150 2500
-F 0 "#PWR0115" H 2150 2350 50  0001 C CNN
-F 1 "+5V" H 2165 2673 50  0000 C CNN
-F 2 "" H 2150 2500 50  0001 C CNN
-F 3 "" H 2150 2500 50  0001 C CNN
-	1    2150 2500
-	1    0    0    -1
-$EndComp
-Wire Wire Line
-	2150 2500 2150 2550
-Wire Wire Line
-	2150 2550 2550 2550
+P 2150 2050
+F 0 "#PWR0115" H 2150 1900 50  0001 C CNN
+F 1 "+5V" H 2165 2223 50  0000 C CNN
+F 2 "" H 2150 2050 50  0001 C CNN
+F 3 "" H 2150 2050 50  0001 C CNN
+	1    2150 2050
+	1    0    0    -1
+$EndComp
+Wire Wire Line
+	2150 2050 2150 2100
+Wire Wire Line
+	2150 2100 2550 2100
 $Comp
 L power:GND #PWR0116
 U 1 1 63D9F245
-P 2700 3500
-F 0 "#PWR0116" H 2700 3250 50  0001 C CNN
-F 1 "GND" H 2705 3327 50  0000 C CNN
-F 2 "" H 2700 3500 50  0001 C CNN
-F 3 "" H 2700 3500 50  0001 C CNN
-	1    2700 3500
-	1    0    0    -1
-$EndComp
-Wire Wire Line
-	2700 3350 2550 3350
-Wire Wire Line
-	2700 3350 2700 3500
+P 2700 3050
+F 0 "#PWR0116" H 2700 2800 50  0001 C CNN
+F 1 "GND" H 2705 2877 50  0000 C CNN
+F 2 "" H 2700 3050 50  0001 C CNN
+F 3 "" H 2700 3050 50  0001 C CNN
+	1    2700 3050
+	1    0    0    -1
+$EndComp
+Wire Wire Line
+	2700 2900 2550 2900
+Wire Wire Line
+	2700 2900 2700 3050
 $Comp
 L power:PWR_FLAG #FLG0101
@@
 F 0 "D1" H 1300 3533 50  0000 C CNN
 F 1 "D" H 1300 3624 50  0000 C CNN
-F 2 "Diode_THT:D_5W_P12.70mm_Horizontal" H 1300 3750 50  0001 C CNN
+F 2 "Diode_THT:D_A-405_P10.16mm_Horizontal" H 1300 3750 50  0001 C CNN
 F 3 "~" H 1300 3750 50  0001 C CNN
 	1    1300 3750
@@
 F 0 "C3" H 1615 3996 50  0000 L CNN
 F 1 "C" H 1615 3905 50  0000 L CNN
-F 2 "Capacitor_THT:CP_Radial_D10.0mm_P5.00mm" H 1538 3800 50  0001 C CNN
+F 2 "Capacitor_THT:C_Radial_D6.3mm_H11.0mm_P2.50mm" H 1538 3800 50  0001 C CNN
 F 3 "~" H 1500 3950 50  0001 C CNN
 	1    1500 3950
@@
 Wire Wire Line
 	1500 4100 1500 4150
+Connection ~ 1500 4150
+Wire Wire Line
+	1500 4150 1650 4150
+$Comp
+L Device:D D3
+U 1 1 63385B64
+P 1100 2900
+F 0 "D3" H 1100 2800 50  0000 C CNN
+F 1 "TVSS" H 1100 3000 50  0000 C CNN
+F 2 "Diode_THT:D_A-405_P10.16mm_Horizontal" H 1100 2900 50  0001 C CNN
+F 3 "~" H 1100 2900 50  0001 C CNN
+	1    1100 2900
+	0    -1   -1   0
+$EndComp
+$Comp
+L Device:D D4
+U 1 1 633B4EB1
+P 1400 2900
+F 0 "D4" H 1400 2800 50  0000 C CNN
+F 1 "TVSS" H 1400 3000 50  0000 C CNN
+F 2 "Diode_THT:D_A-405_P10.16mm_Horizontal" H 1400 2900 50  0001 C CNN
+F 3 "~" H 1400 2900 50  0001 C CNN
+	1    1400 2900
+	0    -1   -1   0
+$EndComp
+$Comp
+L Device:D D2
+U 1 1 633CC5A9
+P 1200 2500
+F 0 "D2" H 1200 2283 50  0000 C CNN
+F 1 "TVSS" H 1200 2374 50  0000 C CNN
+F 2 "Diode_THT:D_A-405_P10.16mm_Horizontal" H 1200 2500 50  0001 C CNN
+F 3 "~" H 1200 2500 50  0001 C CNN
+	1    1200 2500
+	0    -1   -1   0
+$EndComp
+Wire Wire Line
+	2050 2400 1850 2400
+Wire Wire Line
+	1000 2300 1000 2600
+Wire Wire Line
+	1000 2600 850  2600
+Wire Wire Line
+	1200 2350 1200 2300
+Connection ~ 1200 2300
+Wire Wire Line
+	1200 2300 1000 2300
+$Comp
+L power:GND #PWR0117
+U 1 1 63414332
+P 1250 3100
+F 0 "#PWR0117" H 1250 2850 50  0001 C CNN
+F 1 "GND" H 1255 2927 50  0000 C CNN
+F 2 "" H 1250 3100 50  0001 C CNN
+F 3 "" H 1250 3100 50  0001 C CNN
+	1    1250 3100
+	1    0    0    -1
+$EndComp
+Wire Wire Line
+	1850 2400 1850 2300
+Wire Wire Line
+	1200 2300 1700 2300
+Wire Wire Line
+	2050 2600 1850 2600
+Wire Wire Line
+	1850 2600 1850 2700
+Wire Wire Line
+	1850 2700 1700 2700
+Wire Wire Line
+	1200 2650 1200 2700
+Connection ~ 1200 2700
+Wire Wire Line
+	1200 2700 1100 2700
+Wire Wire Line
+	1100 2700 1100 2750
+Connection ~ 1100 2700
+Wire Wire Line
+	1100 2700 850  2700
+Wire Wire Line
+	1400 2700 1400 2750
+Connection ~ 1400 2700
+Wire Wire Line
+	1400 2700 1200 2700
+Wire Wire Line
+	1400 3050 1250 3050
+Wire Wire Line
+	1250 3100 1250 3050
+Connection ~ 1250 3050
+Wire Wire Line
+	1250 3050 1100 3050
+Wire Notes Line
+	1800 4500 1800 1850
+Wire Notes Line
+	1800 1850 550  1850
+Wire Notes Line
+	600  4500 1800 4500
+$Comp
+L Device:R_Small R9
+U 1 1 63544C21
+P 1700 2500
+F 0 "R9" H 1800 2550 50  0000 L CNN
+F 1 "150" H 1750 2450 50  0000 L CNN
+F 2 "Resistor_THT:R_Axial_DIN0204_L3.6mm_D1.6mm_P5.08mm_Horizontal" H 1700 2500 50  0001 C CNN
+F 3 "~" H 1700 2500 50  0001 C CNN
+	1    1700 2500
+	-1   0    0    1
+$EndComp
+Wire Wire Line
+	1700 2400 1700 2300
+Connection ~ 1700 2300
+Wire Wire Line
+	1700 2300 1850 2300
+Wire Wire Line
+	1700 2600 1700 2700
+Connection ~ 1700 2700
+Wire Wire Line
+	1700 2700 1400 2700
 Wire Bus Line
 	6450 3250 6450 3500
@@
 Wire Bus Line
 	9700 1250 9700 3450
-Connection ~ 1500 4150
-Wire Wire Line
-	1500 4150 1650 4150
 $EndSCHEMATC

Commit message: Finish PCB layputting of HP controller
Parts:
- removed R8: 4.7k, Resistor_THT:R_Axial_DIN0204_L3.6mm_D1.6mm_P5.08mm_Horizontal, symbol Device:R_Small
- renumbered R9 to R8
Changed lines of the file:
@@
 Text Label 8250 6150 2    50   ~ 0
 LT
-Text GLabel 6150 3950 2    50   Input ~ 0
+Text GLabel 6250 3950 2    50   Input ~ 0
 RXD
-Text GLabel 6150 4050 2    50   Input ~ 0
+Text GLabel 6250 4050 2    50   Input ~ 0
 TXD
 Wire Wire Line
@@
 	4850 3050 4850 3000
 Wire Wire Line
-	4850 2800 4850 2750
-Wire Wire Line
-	4850 2750 5500 2750
-Wire Wire Line
 	4800 2700 4800 2750
-Wire Wire Line
-	4800 2750 4850 2750
-Connection ~ 4850 2750
-$Comp
-L Device:R_Small R8
-U 1 1 63927284
-P 4850 2900
-F 0 "R8" H 4950 2950 50  0000 L CNN
-F 1 "4.7k" H 4900 2850 50  0000 L CNN
-F 2 "Resistor_THT:R_Axial_DIN0204_L3.6mm_D1.6mm_P5.08mm_Horizontal" H 4850 2900 50  0001 C CNN
-F 3 "~" H 4850 2900 50  0001 C CNN
-	1    4850 2900
-	-1   0    0    1
-$EndComp
 Wire Wire Line
 	8150 1400 8150 1450
@@
 Text Label 8550 4300 2    50   ~ 0
 C_DSET
-Wire Wire Line
-	6100 3950 6150 3950
-Wire Wire Line
-	6100 4050 6150 4050
 Wire Wire Line
 	6300 3450 6100 3450
@@
 Entry Wire Line
 	6350 4550 6450 4650
-Wire Wire Line
-	6150 4150 6100 4150
 $Comp
 L Connector:Screw_Terminal_01x02 J13
@@
 Wire Notes Line
 	10300 3000 10300 500
-Text GLabel 6150 4150 2    50   Input ~ 0
+Text GLabel 6250 4150 2    50   Input ~ 0
 DRIVE
 Text GLabel 3300 2300 2    50   Input ~ 0
@@
 	600  4500 1800 4500
 $Comp
-L Device:R_Small R9
+L Device:R_Small R8
 U 1 1 63544C21
 P 1700 2500
-F 0 "R9" H 1800 2550 50  0000 L CNN
+F 0 "R8" H 1800 2550 50  0000 L CNN
 F 1 "150" H 1750 2450 50  0000 L CNN
 F 2 "Resistor_THT:R_Axial_DIN0204_L3.6mm_D1.6mm_P5.08mm_Horizontal" H 1700 2500 50  0001 C CNN
@@
 Wire Wire Line
 	1700 2700 1400 2700
+Wire Wire Line
+	4800 2750 5500 2750
+Wire Wire Line
+	6100 4150 6250 4150
+Wire Wire Line
+	6100 3950 6250 3950
+Wire Wire Line
+	6100 4050 6250 4050
 Wire Bus Line
 	6450 3250 6450 3500

Commit message: Fix schematic
Parts:
- U1: symbol MCU_Microchip_8051:AT89C4051-24PU -> HP_device-rescue:AT89C4051-24PU-MCU_Microchip_8051
- U2: symbol RS485Device:MCP4162-104 -> HP_device-rescue:MCP4162-104-RS485Device
- U3: symbol RS485Device:MCP4162-503 -> HP_device-rescue:MCP4162-503-RS485Device
- U5: symbol RS485Device:SN65176BP -> HP_device-rescue:SN65176BP-RS485Device
